Commit message: pre-store before arm dof change

File: mm_assets/stretch/stretch_ctrl.urdf (robot description, URDF)
Before this commit: robot stretch, 61 links, 60 joints
Joints:
- joint joint_arm_l0: mimic (none) -> joint=joint_arm_l3 multiplier=1.0 offset=0.0
- joint joint_arm_l1: mimic (none) -> joint=joint_arm_l3 multiplier=1.0 offset=0.0
- joint joint_arm_l2: mimic (none) -> joint=joint_arm_l3 multiplier=1.0 offset=0.0

File: mm_assets/stretch/stretch_sim.urdf (robot description, URDF)
Before this commit: robot stretch, 64 links, 63 joints
Joints:
- joint joint_arm_l0: mimic (none) -> joint=joint_arm_l3 multiplier=1.0 offset=0.0
- joint joint_arm_l1: mimic (none) -> joint=joint_arm_l3 multiplier=1.0 offset=0.0
- joint joint_arm_l2: mimic (none) -> joint=joint_arm_l3 multiplier=1.0 offset=0.0
